File: SSTdriver.kicad_pcb (KiCad board)
At the start: 4 copper layers, 47.3 x 56 mm, 67 parts, among them P1 CONN_01X05, P2 USB_OTG, P3 CONN_01X04, Q1 Fairchild_BCV27, Q2 QRE1113, Q3 DMG3415U-7, Q4 DMG3415U-7, U1 ATMEGA328P-A, U2 FT231X, U3 LMV358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

Commit message: Bom updates mainly, added start of guideport.
Other:
- board text added: "StarSync Trackers Driver v2.2.1"
- board text removed: "StarSync Trackers Driver v2.2.0"
